Commit message: Added left gripper (vacuum gripper) to collision model

File: baxter_description/urdf/baxter_grippers.urdf (robot description, URDF)
Before this commit: robot baxter, 51 links, 50 joints
Links:
- added link left_finger; collision cylinder length=0.11 radius=0.01
Joints:
- added joint left_finger_joint: type fixed, parent left_gripper, child left_finger, origin xyz=0 0 0.01 rpy=0 -0 0, axis 0 0 0
